File: mikroBUS/MikroBusSilToDil.sch (EAGLE design)
At the start: 4 parts

Commit message: 
Parts:
- removed U$3, U$4: MIKROBUS_SIL2, lieven:MIKROBUS_SIL2
Changed lines of the file:
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@@
 <layer number="56" name="wert" color="7" fill="1" visible="no" active="no"/>
 <layer number="57" name="tCAD" color="7" fill="1" visible="no" active="no"/>
+<layer number="59" name="tCarbon" color="7" fill="1" visible="no" active="no"/>
+<layer number="60" name="bCarbon" color="7" fill="1" visible="no" active="no"/>
 <layer number="91" name="Nets" color="2" fill="1" visible="yes" active="yes"/>
 <layer number="92" name="Busses" color="1" fill="1" visible="yes" active="yes"/>
@@
 <layer number="127" name="_tValues" color="7" fill="1" visible="yes" active="yes"/>
 <layer number="128" name="_bValues" color="7" fill="1" visible="yes" active="yes"/>
+<layer number="129" name="Mask" color="7" fill="1" visible="yes" active="yes"/>
 <layer number="131" name="tAdjust" color="7" fill="1" visible="no" active="yes"/>
 <layer number="132" name="bAdjust" color="7" fill="1" visible="no" active="yes"/>
@@
 <parts>
 <part name="U$1" library="lieven" deviceset="MIKROBUS" device="900MIL"/>
-<part name="U$3" library="lieven" deviceset="MIKROBUS_SIL2" device=""/>
-<part name="U$4" library="lieven" deviceset="MIKROBUS_SIL2" device=""/>
 <part name="U$5" library="lieven" deviceset="MIKROBUS" device="SIL"/>
 </parts>
